File: Lidar_w:Encoders/Lidar_w:Encoders.kicad_pcb (KiCad board)
At the start: 2 copper layers, 67 x 61.5 mm, 15 parts, among them J1 DB15_HighDensity_MountingHoles, J2 DB15_HighDensity_MountingHoles, P1 CONN_01X04, P2 CONN_01X04, P3 CONN_01X04, P4 CONN_01X04, P5 CONN_01X05, P6 CONN_01X04, U1 MCP2551-I/P, U2 Teensy3.6

Commit message: added extra grounds
Routing:
- net GND: track 18.3 -> 38.2 mm
Changed lines of the file:
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@@
   (general
     (links 62)
-    (no_connects 3)
+    (no_connects 2)
     (area 148.924999 75.146999 216.075001 143.385)
     (thickness 1.6)
     (drawings 11)
-    (tracks 258)
+    (tracks 268)
     (zones 0)
     (modules 15)
@@
   (gr_line (start 216 81.5) (end 216 140.5) (angle 90) (layer Edge.Cuts) (width 0.15))
   (gr_line (start 215 81.5) (end 216 81.5) (angle 90) (layer Edge.Cuts) (width 0.15))
-  (segment (start 191.525 93) (end 193.815 93) (width 1) (layer B.Cu) (net 1) (status C00000))
-  (segment (start 193.815 93) (end 196.105 93) (width 1) (layer B.Cu) (net 1) (status C00000))
-  (segment (start 196.105 93) (end 198.395 93) (width 1) (layer B.Cu) (net 1) (status C00000))
-  (segment (start 198.395 93) (end 200.685 93) (width 1) (layer B.Cu) (net 1) (status C00000))
-  (segment (start 160.525 93) (end 162.815 93) (width 1) (layer B.Cu) (net 1) (status C00000))
-  (segment (start 162.815 93) (end 165.105 93) (width 1) (layer B.Cu) (net 1) (status C00000))
-  (segment (start 165.105 93) (end 167.395 93) (width 1) (layer B.Cu) (net 1) (status C00000))
-  (segment (start 167.395 93) (end 169.685 93) (width 1) (layer B.Cu) (net 1) (status C00000))
+  (segment (start 188 110.5) (end 188 108.890001) (width 1) (layer B.Cu) (net 1) (status 800000))
+  (segment (start 188 108.890001) (end 188.375001 108.515) (width 1) (layer B.Cu) (net 1) (status C00000))
+  (segment (start 191.525 93) (end 189 93) (width 1) (layer F.Cu) (net 1) (status 400000))
+  (segment (start 191.525 93) (end 193.815 93) (width 1) (layer F.Cu) (net 1) (status C00000))
+  (segment (start 196.105 93) (end 193.815 93) (width 1) (layer F.Cu) (net 1) (status C00000))
+  (segment (start 196.105 93) (end 198.395 93) (width 1) (layer F.Cu) (net 1) (status C00000))
+  (segment (start 200.685 93) (end 198.395 93) (width 1) (layer F.Cu) (net 1) (status C00000))
+  (segment (start 203 93) (end 200.685 93) (width 1) (layer F.Cu) (net 1) (status 800000))
+  (segment (start 162.815 93) (end 160.525 93) (width 1) (layer F.Cu) (net 1) (status C00000))
+  (segment (start 165.105 93) (end 162.815 93) (width 1) (layer F.Cu) (net 1) (status C00000))
+  (segment (start 167.395 93) (end 165.105 93) (width 1) (layer F.Cu) (net 1) (status C00000))
+  (segment (start 169.685 93) (end 167.395 93) (width 1) (layer F.Cu) (net 1) (status C00000))
+  (segment (start 169.685 93) (end 173 93) (width 1) (layer F.Cu) (net 1) (status 400000))
+  (segment (start 160.525 93) (end 158.5 93) (width 1) (layer F.Cu) (net 1) (status 400000))
+  (segment (start 158.5 93) (end 158 93.5) (width 1) (layer F.Cu) (net 1))
+  (segment (start 160.525 93) (end 162.815 93) (width 1) (layer B.Cu) (net 1))
+  (segment (start 162.815 93) (end 165.105 93) (width 1) (layer B.Cu) (net 1))
+  (segment (start 165.105 93) (end 167.395 93) (width 1) (layer B.Cu) (net 1))
   (segment (start 192 135) (end 192 136.5) (width 0.65) (layer B.Cu) (net 2) (status 10))
   (segment (start 199.54 136.46) (end 199.54 135) (width 0.65) (layer B.Cu) (net 2) (status 20))
