File: Lidar_w-Encoders/Lidar_w-Encoders.sch (KiCad schematic (older format))
At the start: 20 parts, among them J1 DB15_HighDensity_MountingHoles, J2 DB15_HighDensity_MountingHoles, P1 CONN_01X04, P10 CONN_01X04, P11 CONN_01X04, P2 CONN_01X04, P3 CONN_01X04, P4 CONN_01X04, P5 CONN_01X05, P6 CONN_01X04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

Commit message: added connector labels and cleaned up
Parts:
- removed P8: CONN_01X04, Socket_Strips:Socket_Strip_Straight_1x04_Pitch2.54mm, symbol CONN_01X04
Connections:
- net CANH: now also P7.4 (P4)
- net CANL: now also P7.5 (P5)
- net CAN_Rx: no longer P7.5 (P5)
- net CAN_Tx: no longer P7.4 (P4)
Changed lines of the file:
@@
 Wire Wire Line
 	8200 4500 8050 4500
-$Comp
-L CONN_01X04 P8
-U 1 1 58C353A8
-P 4750 4850
-F 0 "P8" H 4750 5100 50  0000 C CNN
-F 1 "CONN_01X04" V 4850 4850 50  0000 C CNN
-F 2 "Socket_Strips:Socket_Strip_Straight_1x04_Pitch2.54mm" H 4750 4850 50  0001 C CNN
-F 3 "" H 4750 4850 50  0000 C CNN
-	1    4750 4850
-	1    0    0    -1
-$EndComp
-$Comp
-L +12V #PWR043
-U 1 1 58C353AE
-P 4550 4700
-F 0 "#PWR043" H 4550 4550 50  0001 C CNN
-F 1 "+12V" H 4550 4840 50  0000 C CNN
-F 2 "" H 4550 4700 50  0000 C CNN
-F 3 "" H 4550 4700 50  0000 C CNN
-	1    4550 4700
-	0    -1   -1   0
-$EndComp
-$Comp
-L GND #PWR044
-U 1 1 58C353B4
-P 4550 4800
-F 0 "#PWR044" H 4550 4550 50  0001 C CNN
-F 1 "GND" H 4550 4650 50  0000 C CNN
-F 2 "" H 4550 4800 50  0000 C CNN
-F 3 "" H 4550 4800 50  0000 C CNN
-	1    4550 4800
-	0    1    1    0
-$EndComp
-$Comp
-L GND #PWR045
-U 1 1 58C353BA
-P 4550 4900
-F 0 "#PWR045" H 4550 4650 50  0001 C CNN
-F 1 "GND" H 4550 4750 50  0000 C CNN
-F 2 "" H 4550 4900 50  0000 C CNN
-F 3 "" H 4550 4900 50  0000 C CNN
-	1    4550 4900
-	0    1    1    0
-$EndComp
-$Comp
-L +5V #PWR046
-U 1 1 58C353C0
-P 4550 5000
-F 0 "#PWR046" H 4550 4850 50  0001 C CNN
-F 1 "+5V" H 4550 5140 50  0000 C CNN
-F 2 "" H 4550 5000 50  0000 C CNN
-F 3 "" H 4550 5000 50  0000 C CNN
-	1    4550 5000
-	0    -1   -1   0
-$EndComp
 Wire Wire Line
 	7450 5600 7550 5600
@@
 	0    -1   -1   0
 $EndComp
-Text Label 8050 4400 0    60   ~ 0
-CAN_Tx
-Text Label 8050 4500 0    60   ~ 0
-CAN_Rx
 $Comp
 L CONN_01X04 P9
@@
 	0    1    1    0
 $EndComp
+Text Label 8050 4400 0    60   ~ 0
+CANH
+Text Label 8050 4500 0    60   ~ 0
+CANL
 $EndSCHEMATC

Commit message: changes
Parts:
- added P8: CONN_01X04, Socket_Strips:Socket_Strip_Straight_1x04_Pitch2.54mm, symbol CONN_01X04
Connections:
- net +5V: now also P8.3 (P3)
- net A1: now also P1.1 (P1); no longer P1.2 (P2)
- net A2: now also P2.1 (P1); no longer P2.2 (P2)
- net A3: now also P8.1 (P1); no longer P3.1 (P1)
- net A4: now also P3.1 (P1); no longer P4.1 (P1)
- net A5: now also P4.1 (P1); no longer P10.1 (P1)
- net A6: now also P10.1 (P1); no longer P11.1 (P1)
- net A7: now also P11.1 (P1); no longer P9.1 (P1)
- net B1: now also P1.2 (P2); no longer P1.1 (P1)
- net B2: now also P2.2 (P2); no longer P2.1 (P1)
- net B3: now also P8.2 (P2); no longer P3.2 (P2)
- net B4: now also P3.2 (P2); no longer P4.2 (P2)
- net B5: now also P4.2 (P2); no longer P10.2 (P2)
- net B6: now also P10.2 (P2); no longer P11.2 (P2)
- net B7: now also P11.2 (P2); no longer P9.2 (P2)
- net GND: now also P8.4 (P4)
- net A8: now reaches U2.13 (11_MOSI0)
- net A8: now also P9.1 (P1)
- net B8: now reaches U2.14 (12_MISO0)
- net B8: now also P9.2 (P2)
